File: licznik/licznik.kicad_pcb (KiCad board)
At the start: 2 copper layers, 72 x 44.1 mm, 66 parts, among them J4 1140084168, J5 Conn_01x03_Female, U1 AMS1117-3.3, U2 AMS1117-5.0, U6 oled, Y1 Crystal

Commit message: wip
Other:
- net class Default removed

Commit message: hardware_2
Parts:
- removed  LSM6DS3: gyro, licznik:gy1
- removed DEBUG UART: Conn_01x03_Female, Connector_PinSocket_2.54mm:PinSocket_1x03_P2.54mm_Vertical
- removed GPS NEO-6M: gps, licznik:gp1
- removed INPUT: Conn_01x04_Female, Connector_PinSocket_2.54mm:PinSocket_1x04_P2.54mm_Vertical
- removed J4: 1140084168, licznik:AMPHENOL_1140084168
- removed J5: Conn_01x03_Female, Connector_PinSocket_2.54mm:PinSocket_1x03_P2.54mm_Vertical
- removed PB_DOWN1, PB_UP1: SW_Push, Connector_PinSocket_2.54mm:PinSocket_2x01_P2.54mm_Vertical
- removed PM_OK1: PB_OK, Connector_PinSocket_2.54mm:PinSocket_2x01_P2.54mm_Vertical
- removed PROG: Conn_01x05_Female, Connector_PinSocket_2.54mm:PinSocket_1x05_P2.54mm_Vertical
- removed R17: 510R, Resistor_SMD:R_0805_2012Metric
- removed RESET1: SW_Push, Button_Switch_THT:SW_PUSH_6mm
- removed STM32F407VET6: STM32F407VETx, Package_QFP:LQFP-100_14x14mm_P0.5mm
- removed Z1, Z2: KDZ3.3V-RTK/P, Diode_SMD:D_SOT-23_ANK
- added B+: BAT+, Connector_PinHeader_2.54mm:PinHeader_1x01_P2.54mm_Vertical, F.Cu at (123.1, 71.7)
- added B-: BAT-, Connector_PinHeader_2.54mm:PinHeader_1x01_P2.54mm_Vertical, F.Cu at (119.1, 71.6)
- added C25: 10uF, Capacitor_SMD:C_0603_1608Metric, F.Cu at (126.8, 71.3)
- added C26: 22uF, Capacitor_SMD:C_0603_1608Metric, F.Cu at (140.8, 109.7)
- added C27: 22uF, Capacitor_SMD:C_0603_1608Metric, F.Cu at (140.8, 104.5)
- added D8: LED, LED_SMD:LED_0603_1608Metric, F.Cu at (138.4, 102.1)
- added H1: MountingHole_Pad, MountingHole:MountingHole_3.2mm_M3, F.Cu at (179.2, 70.5)
- added H2: MountingHole_Pad, MountingHole:MountingHole_3.2mm_M3, F.Cu at (111.2, 70.4)
- added H3: MountingHole_Pad, MountingHole:MountingHole_3.2mm_M3, F.Cu at (179.3, 109.8)
- added H4: MountingHole_Pad, MountingHole:MountingHole_3.2mm_M3, F.Cu at (111.2, 109.7)
- added J2: USB_B_Mini, Connector_USB:USB_Mini-B_Wuerth_65100516121_Horizontal, F.Cu at (121.8, 105.3)
- added LEN_ON: jump, Connector_PinHeader_1.00mm:PinHeader_1x02_P1.00mm_Vertical, F.Cu at (135.7, 99.2)
- added MICRO_SD: TF-01A, slot_sd:TF-01A, F.Cu at (173.9, 83.0)
- added PB_POWER: POWER_PB, Connector_PinSocket_2.54mm:PinSocket_2x01_P2.54mm_Vertical, F.Cu at (135.3, 103.7)
- added PB_UP: SW_Push, Connector_PinSocket_2.54mm:PinSocket_2x01_P2.54mm_Vertical, F.Cu at (158.8, 70.6)
- added Q1: AO3401A, Package_TO_SOT_SMD:SOT-23, F.Cu at (130.7, 71.1)
- added R20: 2K, Resistor_SMD:R_0603_1608Metric, F.Cu at (138.0, 74.8)
- added R21: 0.1R, Resistor_SMD:R_0603_1608Metric, F.Cu at (134.7, 71.2)
- added R23: 10K, Resistor_SMD:R_0603_1608Metric, F.Cu at (111.5, 77.9)
- added R24: 2K, Resistor_SMD:R_0603_1608Metric, F.Cu at (138.4, 105.5)
- added RESET: USER_PB, TS_1187A-B-A-B:SW_TS-1187A-B-A-B, F.Cu at (166.5, 106.3)
- added SWD: Conn_01x05_Female, Connector_PinSocket_2.54mm:PinSocket_1x05_P2.54mm_Vertical, F.Cu at (163.4, 70.8)
- added U3: STM32F407VETx, Package_QFP:LQFP-100_14x14mm_P0.5mm, F.Cu at (144.1, 89.2)
- added U4: gps, licznik:gp1, F.Cu at (176.7, 99.7)
- added U5: gyro, licznik:gy1, F.Cu at (165.3, 101.2)
- added U8: TP4056, Package_SO:HSOP-8-1EP_3.9x4.9mm_P1.27mm_EP2.3x2.3mm, F.Cu at (125.4, 76.7)
- C1, C11, C12, C13, C14, C15, C16, C17, C18, C19, C2, C20, C21, C22, C23, C3, C4, C5, C6: footprint Capacitor_SMD:C_0805_2012Metric -> Capacitor_SMD:C_0603_1608Metric
- C10, C8: value 10uF -> 100nF; footprint Capacitor_Tantalum_SMD:CP_EIA-3216-18_Kemet-A -> Capacitor_SMD:C_0603_1608Metric
- D2: footprint LED_SMD:LED_0805_2012Metric -> LED_SMD:LED_0603_1608Metric; moved to F.Cu
- D3: value LED -> SM4007; footprint LED_SMD:LED_0805_2012Metric -> Diode_SMD:D_SOD-123F; moved to F.Cu
- D4: value LED -> ZMMxx; footprint LED_SMD:LED_0805_2012Metric -> Diode_SMD:D_MiniMELF
- F1: footprint Fuse:Fuse_0805_2012Metric -> Diode_SMD:D_SMB
- R1, R10, R11, R12, R13, R15, R16, R18, R2, R3, R4, R5, R8, R9: footprint Resistor_SMD:R_0805_2012Metric -> Resistor_SMD:R_0603_1608Metric
- R14: value 510R -> 0R; footprint Resistor_SMD:R_0805_2012Metric -> Resistor_SMD:R_0603_1608Metric
- R6, R7: value 510R -> 10K; footprint Resistor_SMD:R_0805_2012Metric -> Resistor_SMD:R_0603_1608Metric
- U2: value AMS1117-5.0 -> LSM6DS3; footprint Package_TO_SOT_SMD:SOT-223-3_TabPin2 -> Package_LGA:LGA-14_3x2.5mm_P0.5mm_LayoutBorder3x4y
- moved R7 69.7 mm to (161.2, 73.6), turned to 0 degrees
- moved C10 54.5 mm to (145.8, 109.7), turned to 0 degrees
- moved C19 52.0 mm to (147.7, 72.0)
- moved U2 51.2 mm to (144.8, 104.5)
- moved C22 50.7 mm to (151.4, 72.0)
- moved C8 50.4 mm to (145.8, 107.2), turned to 180 degrees
- moved C21 45.8 mm to (151.3, 74.5)
- moved C18 44.9 mm to (140.7, 72.1), turned to 180 degrees
- moved C17 43.5 mm to (144.2, 72.1)
- moved C16 40.0 mm to (144.2, 74.5)
- moved C20 37.9 mm to (147.8, 74.5)
- moved C15 36.8 mm to (135.6, 74.8), turned to 90 degrees
- moved R14 36.7 mm to (147.6, 100.1), turned to -90 degrees
- moved FB1 33.6 mm to (132.2, 100.2), turned to 90 degrees
- moved F1 33.0 mm to (131.2, 107.0)
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Connections:
- C10 pad 1: +5V -> GND
- C10 pad 2: GND -> +3V3
- C7 pad 1: Net-(C7-Pad1) -> REG_IN
- C8 pad 1: Net-(C7-Pad1) -> +3V3
- D1 pad 2: +12V -> Net-(D1-A)
- D2 pad 2: Net-(D2-Pad2) -> Net-(D2-A)
- D3 pad 1: LED_2 -> REG_IN
- D3 pad 2: Net-(D3-Pad2) -> +5V
- D4 pad 1: GND -> +5V
- D4 pad 2: Net-(D4-Pad2) -> GND
- FB1 pad 1: Net-(C7-Pad1) -> Net-(FB1-Pad1)
- R11 pad 1: SDIO_D0 -> SDIO_D3
- R12 pad 1: SDIO_D1 -> SDIO_CMD
- R13 pad 1: SDIO_CMD -> SDIO_SCK
- R14 pad 1: Net-(J3-Pad3) -> Net-(D2-A)
- R14 pad 2: ENGINE_RPM_INPUT -> Net-(R14-Pad2)
- R15 pad 1: SDIO_SCK -> SDIO_D0
- R16 pad 1: SDIO_D3 -> SDIO_D1
- R5 pad 1: Net-(D2-Pad2) -> Net-(R14-Pad2)
- R6 pad 1: Net-(D3-Pad2) -> CHRG_SIGNAL
- R7 pad 1: Net-(D4-Pad2) -> SDIO_INSERT_CARD
- U1 pad 3: Net-(C7-Pad1) -> REG_IN
- U2 pad 1: GND -> GYRO_MISO
- U2 pad 2: +5V -> GND
- U2 pad 3: Net-(C7-Pad1) -> GND
Routing:
- net REG_IN: track 0.00 -> 145.0 mm
- net GND: track 373.0 -> 443.6 mm, vias 2 -> 6
- net SDIO_INSERT_CARD: track 0.00 -> 56.5 mm
- net +3V3: track 356.6 -> 308.7 mm, vias 3 -> 7
- net Net-(C7-Pad1): track 38.0 -> 0.00 mm
- net CHRG_SIGNAL: track 0.00 -> 37.4 mm, vias 0 -> 2
- net GYRO_MISO: track 17.0 -> 51.4 mm, vias 1 -> 0
- net PB_OK: track 70.1 -> 36.3 mm
- net +5V: track 82.0 -> 111.1 mm, vias 1 -> 2
- net WHEEL_RPM_INPUT: track 27.7 -> 0.00 mm
- net ENGINE_RPM_INPUT: track 26.0 -> 0.00 mm
- net Net-(D1-K): track 2.81 -> 27.9 mm
- net PB_DOWN: track 55.0 -> 31.3 mm, vias 2 -> 0
- net Net-(U3-VCAP_2): track 25.1 -> 2.97 mm, vias 2 -> 0
- net OLED_SCK: track 63.3 -> 41.2 mm, vias 0 -> 1
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Other:
- board size 72 x 44.1 mm -> 72 x 43.2 mm
- board text added: "GPS"
- board text added: "Gnd"
- board text added: "Rx"
- board text added: "Tx"
- board text added: "Vcc"
- board text removed: "12V"
- board text removed: "GND"
- board text removed: "Grzegorz W Licznik Motocyklowy"
- board text removed: "rpm"
- board text removed: "speed"

Commit message: ulepszony pcb
Parts:
- moved FB1 0.28 mm to (132.4, 100.2)
Changed lines of the file:
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@@
   )
   (footprint "Inductor_SMD:L_0805_2012Metric" (layer "F.Cu")
-    (at 132.1562 100.1776 90)
+    (at 132.4356 100.203 90)
     (descr "Inductor SMD 0805 (2012 Metric), square (rectangular) end terminal, IPC_7351 nominal, (Body size source: IPC-SM-782 page 80, https://www.pcb-3d.com/wordpress/wp-content/uploads/ipc-sm-782a_amendment_1_and_2.pdf), generated with kicad-footprint-generator")
     (tags "inductor")

Commit message: wip
Parts:
- removed RESET: USER_PB, TS_1187A-B-A-B:SW_TS-1187A-B-A-B
- removed U4: gps, licznik:gp1
- removed U5: gyro, licznik:gy1
- added GPS1: GPS, BM04B-SRSS-TB_LF__SN_:JST_BM04B-SRSS-TB_LF__SN_, B.Cu at (170.5, 107.0)
- added J3: BAT+, Connector_PinHeader_2.54mm:PinHeader_1x01_P2.54mm_Vertical, F.Cu at (95.7, 57.1)
- added J4: BAT-, Connector_PinHeader_2.54mm:PinHeader_1x01_P2.54mm_Vertical, F.Cu at (95.7, 61.8)
- added RADIO1: NRF24L01_Breakout, nRF:NRF24L01-SMD_mini, F.Cu at (170.0, 98.5)
- added USER_PB1: USER_PB, TS_1187A-B-A-B:SW_TS-1187A-B-A-B, F.Cu at (162.5, 108.0)
Connections:
- C11 pad 1: Net-(U3-VCAP_1) -> Net-(CPU1-VCAP_1)
- C13 pad 1: Net-(U3-VCAP_2) -> Net-(CPU1-VCAP_2)
- C27 pad 1: +3V3 -> REG_OUT
- C9 pad 1: +3V3 -> REG_OUT
- FB1 pad 1: Net-(FB1-Pad1) -> +5V
- FB1 pad 2: Net-(F1-Pad2) -> Net-(D1-K)
- J2 pad 2: PB_OK -> REG_OUT
- J2 pad 4: GND -> +3V3
- R6 pad 2: +3V3 -> +5V
- R8 pad 2: Net-(U3-BOOT0) -> Net-(CPU1-BOOT0)
- R9 pad 2: Net-(U3-PB2) -> Net-(CPU1-PB2)
- U1 pad 2: +3V3 -> REG_OUT
- U3 pad 67: unconnected-(U3-PA8-Pad67) -> nRF24_CE
- U3 pad 68: unconnected-(U3-PA9-Pad68) -> nRF24_IRQ
- U3 pad 69: unconnected-(U3-PA10-Pad69) -> nRF24_CNS
Routing:
- net GND: track 443.6 -> 384.4 mm, vias 6 -> 5
- net NRST: track 90.9 -> 35.9 mm, vias 3 -> 1
- net GYRO_MISO: track 51.4 -> 5.75 mm
- net REG_IN: track 145.0 -> 102.1 mm
- net GYRO_SCK: track 44.4 -> 3.25 mm, vias 1 -> 0
- net GYRO_MOSI: track 43.4 -> 4.21 mm, vias 1 -> 0
- net GPS_UART_TX: track 38.8 -> 0.00 mm
- net GPS_UART_RX: track 32.1 -> 0.00 mm
- net GYRO_CS: track 32.5 -> 7.43 mm
- net +3V3: track 308.7 -> 292.1 mm
- removed copper zone on B.Cu, net GND
- removed copper zone on F.Cu, net GND
Other:
- board text removed: "GPS"
- board text removed: "Gnd"
- board text removed: "Rx"
- board text removed: "Tx"
- board text removed: "Vcc"

Commit message: przed poprawkami
Parts:
- removed B+: BAT+, Connector_PinHeader_2.54mm:PinHeader_1x01_P2.54mm_Vertical
- removed B-: BAT-, Connector_PinHeader_2.54mm:PinHeader_1x01_P2.54mm_Vertical
- removed D8: LED, LED_SMD:LED_0603_1608Metric
- removed F1: Fuse_Small, Diode_SMD:D_SMB
- removed GPS1: GPS, BM04B-SRSS-TB_LF__SN_:JST_BM04B-SRSS-TB_LF__SN_
- removed LEN_ON: jump, Connector_PinHeader_1.00mm:PinHeader_1x02_P1.00mm_Vertical
- removed MICRO_SD: TF-01A, slot_sd:TF-01A
- removed PB_POWER: POWER_PB, Connector_PinSocket_2.54mm:PinSocket_2x01_P2.54mm_Vertical
- removed SWD: Conn_01x05_Female, Connector_PinSocket_2.54mm:PinSocket_1x05_P2.54mm_Vertical
- removed U3: STM32F407VETx, Package_QFP:LQFP-100_14x14mm_P0.5mm
- removed USER_PB1: USER_PB, TS_1187A-B-A-B:SW_TS-1187A-B-A-B
- added CPU1: STM32F407VETx, Package_QFP:LQFP-100_14x14mm_P0.5mm, F.Cu at (145.6, 88.8)
- added J1: Conn_01x05_Female, Connector_PinSocket_2.54mm:PinSocket_1x05_P2.54mm_Vertical, F.Cu at (163.5, 71.1)
- added J5: PRT-14417, BM04B-SRSS-TB_LF__SN_:SPARKFUN_PRT-14417, B.Cu at (155.6, 107.7)
- added J6: Conn_01x02_Pin, Connector_JST:JST_PH_S2B-PH-SM4-TB_1x02-1MP_P2.00mm_Horizontal, B.Cu at (176.1, 100.6)
- added MICRO_SD1: TF-01A, slot_sd:TF-01A, F.Cu at (178.9, 83.4)
- added R17: 0R, Resistor_SMD:R_0603_1608Metric, F.Cu at (171.8, 109.2)
- added R19: 0R, Resistor_SMD:R_0603_1608Metric, F.Cu at (161.4, 87.2)
- added R22: 0R, Resistor_SMD:R_0603_1608Metric, F.Cu at (158.7, 87.2)
- added R25: 0R, Resistor_SMD:R_0603_1608Metric, F.Cu at (162.0, 91.7)
- added R26: 0R, Resistor_SMD:R_0603_1608Metric, F.Cu at (158.3, 109.2)
- added R27: 0R, Resistor_SMD:R_0603_1608Metric, F.Cu at (150.2, 109.3)
- added R28: 0R, Resistor_SMD:R_0603_1608Metric, F.Cu at (155.6, 109.2)
- added R29: 0R, Resistor_SMD:R_0603_1608Metric, F.Cu at (152.9, 109.2)
- added RESET1: RESET, TS_1187A-B-A-B:SW_TS-1187A-B-A-B, F.Cu at (127.0, 74.1)
- R2, R4: value 10K -> 0R
- R24: value 2K -> 0R
- moved R2 48.1 mm to (168.9, 109.2), turned to -90 degrees
- moved R4 41.1 mm to (166.1, 109.2), turned to -90 degrees
- moved R23 38.9 mm to (135.9, 108.2), turned to -90 degrees
- moved Q1 36.9 mm to (131.6, 108.0), turned to 0 degrees
- moved J3 31.6 mm to (120.8, 76.3)
- moved D3 30.5 mm to (139.5, 108.9)
- moved C19 29.6 mm to (139.0, 100.4), turned to 90 degrees
- moved C17 29.3 mm to (136.6, 100.4), turned to 90 degrees
- moved C22 28.4 mm to (152.7, 100.4), turned to -90 degrees
- moved R20 27.4 mm to (115.6, 90.5)
- moved J4 25.8 mm to (117.1, 76.3)
- moved C27 25.8 mm to (115.0, 103.5), turned to -90 degrees
- moved R21 25.6 mm to (118.6, 91.1), turned to 180 degrees
- moved R24 25.1 mm to (163.2, 109.2)
- moved U1 19.3 mm to (123.0, 96.8), turned to 0 degrees
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Connections:
- C26 pad 1: REG_IN -> SW_OUT
- C27 pad 1: REG_OUT -> +3V3
- C7 pad 1: REG_IN -> SW_OUT
- C9 pad 1: REG_OUT -> +3V3
- D3 pad 1: REG_IN -> SW_IN
- J2 pad 2: REG_OUT -> SW_IN
- J2 pad 4: +3V3 -> SW_OUT
- Q1 pad 2: REG_IN -> SW_IN
- R2 pad 1: PB_UP -> Net-(RADIO1-MOSI)
- R2 pad 2: +3V3 -> OLED_MOSI
- R24 pad 1: Net-(D8-A) -> Net-(RADIO1-IRQ)
- R24 pad 2: REG_IN -> nRF24_IRQ
- R4 pad 1: PB_OK -> Net-(RADIO1-MISO)
- R4 pad 2: +3V3 -> OLED_MISO
- RADIO1 pad 2: +3V3 -> Net-(RADIO1-VCC)
- RADIO1 pad 3: nRF24_CE -> Net-(RADIO1-CE)
- RADIO1 pad 4: nRF24_CNS -> Net-(RADIO1-~{CSN})
- RADIO1 pad 5: OLED_SCK -> Net-(RADIO1-SCK)
- RADIO1 pad 6: OLED_MOSI -> Net-(RADIO1-MOSI)
- RADIO1 pad 7: OLED_MISO -> Net-(RADIO1-MISO)
- RADIO1 pad 8: nRF24_IRQ -> Net-(RADIO1-IRQ)
- U1 pad 2: REG_OUT -> +3V3
- U1 pad 3: REG_IN -> SW_OUT
Routing:
- net REG_IN: track 102.1 -> 0.00 mm
- net VBAT: track 14.6 -> 111.4 mm, vias 0 -> 1
- net GND: track 384.4 -> 466.8 mm, vias 5 -> 1
- net +5V: track 111.1 -> 33.9 mm, vias 2 -> 0
- net SW_OUT: track 0.00 -> 75.6 mm
- net +3V3: track 292.1 -> 217.4 mm, vias 7 -> 2
- net OLED_MOSI: track 40.5 -> 106.2 mm, vias 1 -> 4
- net OLED_SCK: track 41.2 -> 105.2 mm, vias 1 -> 4
- net NRST: track 35.9 -> 84.1 mm, vias 1 -> 2
- net OLED_MISO: track 0.00 -> 39.8 mm, vias 0 -> 2
- net nRF24_IRQ: track 0.00 -> 36.9 mm
- net GYRO_MOSI: track 4.21 -> 37.3 mm, vias 0 -> 2
- net PB_OK: track 36.3 -> 5.95 mm, vias 2 -> 0
- net SW_IN: track 0.00 -> 29.0 mm
- net GPS_UART_RX: track 0.00 -> 26.1 mm
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Other:
- board size 72 x 43.2 mm -> 77.3 x 48.3 mm

Commit message: proukcja v5
Parts:
- removed C26, C27: 22uF, Capacitor_SMD:C_0603_1608Metric
- removed C7, C9: 10uF, Capacitor_Tantalum_SMD:CP_EIA-3216-18_Kemet-A
- removed D3: SM4007, Diode_SMD:D_SOD-123F
- removed D4: ZMMxx, Diode_SMD:D_MiniMELF
- removed Q1: AO3401A, Package_TO_SOT_SMD:SOT-23
- removed R14: 0R, Resistor_SMD:R_0603_1608Metric
- removed RESET1: RESET, TS_1187A-B-A-B:SW_TS-1187A-B-A-B
- added L1: 10uH, Inductor_SMD:L_0805_2012Metric, F.Cu at (128.8, 95.0)
- added R30: 120K, Resistor_SMD:R_0603_1608Metric, F.Cu at (129.1, 100.9)
- added R31: 200K, Resistor_SMD:R_0603_1608Metric, F.Cu at (121.7, 101.1)
- C1, C11, C12, C13, C14, C15, C16, C17, C18, C19, C20, C21, C22, C6: footprint Capacitor_SMD:C_0603_1608Metric -> Capacitor_SMD:C_0402_1005Metric
- C2, C5: value 100nF -> 10uF
- C3: value 100nF -> 47pF; footprint Capacitor_SMD:C_0603_1608Metric -> Resistor_SMD:R_1206_3216Metric
- R1: value 10K -> 50K
- R18, R8, R9: footprint Resistor_SMD:R_0603_1608Metric -> Resistor_SMD:R_0402_1005Metric
- R23: value 10K -> 510K
- U1: value AMS1117-3.3 -> MCP1601-I_MS; footprint Package_TO_SOT_SMD:SOT-223-3_TabPin2 -> Package_DFN_QFN:TDFN-8-1EP_3x2mm_P0.5mm_EP1.3x1.4mm
- moved C3 29.1 mm to (125.5, 101.2), turned to 180 degrees
- moved PB_UP 28.1 mm to (131.4, 77.3), turned to 180 degrees
- moved C16 26.5 mm to (140.1, 99.4), turned to 180 degrees
- moved C2 26.2 mm to (121.8, 97.6), turned to -90 degrees
- moved C22 25.4 mm to (139.4, 78.8), turned to 0 degrees
- moved C15 23.7 mm to (140.1, 100.7)
- moved R17 19.9 mm to (159.2, 93.8), turned to 180 degrees
- moved C5 19.2 mm to (125.5, 103.2)
- moved C23 17.1 mm to (160.1, 82.5), turned to -90 degrees
- moved R2 16.6 mm to (159.3, 95.7), turned to 180 degrees
- moved J1 16.3 mm to (147.6, 74.8)
- moved C19 14.3 mm to (136.1, 86.4), turned to -90 degrees
- moved C18 13.0 mm to (134.9, 86.4), turned to -90 degrees
- moved R20 12.8 mm to (128.3, 88.4), turned to -90 degrees
- moved FB1 12.8 mm to (115.7, 95.1), turned to -90 degrees
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Connections:
- C2 pad 1: NRST -> SW_OUT
- C25 pad 1: VBAT -> SW_IN
- C3 pad 1: PB_UP -> +3V3
- C3 pad 2: GND -> Net-(U1-FB)
- C4 pad 1: PB_DOWN -> PUSH_DOWN_IN
- C5 pad 1: PB_OK -> +3V3
- J2 pad 3: PB_DOWN -> PUSH_DOWN_IN
- J3 pad 1: VBAT -> SW_IN
- J6 pad 2: VBAT -> SW_IN
- R1 pad 1: NRST -> PB_DOWN
- R1 pad 2: +3V3 -> PUSH_DOWN_IN
- R23 pad 1: GND -> Net-(R23-Pad1)
- R23 pad 2: +5V -> +3V3
- R3 pad 1: PB_DOWN -> PUSH_DOWN_IN
- R5 pad 1: Net-(R14-Pad2) -> Net-(D2-A)
- R6 pad 2: +5V -> +3V3
- U1 pad 1: GND -> SW_OUT
- U1 pad 2: +3V3 -> SW_OUT
- U1 pad 3: SW_OUT -> Net-(U1-FB)
- U8 pad 5: VBAT -> SW_IN
Routing:
- net GND: track 466.8 -> 196.9 mm, vias 1 -> 24
- net VBAT: track 111.4 -> 0.00 mm, vias 1 -> 0
- net SW_IN: track 29.0 -> 104.7 mm, vias 0 -> 1
- net NRST: track 84.1 -> 40.3 mm, vias 2 -> 1
- net PUSH_DOWN_IN: track 0.00 -> 41.9 mm, vias 0 -> 2
- net PB_DOWN: track 40.8 -> 2.78 mm, vias 2 -> 0
- net +3V3: track 217.4 -> 249.8 mm, vias 2 -> 7
- net +5V: track 33.9 -> 3.87 mm
- net PB_UP: track 39.8 -> 11.5 mm
- net SW_OUT: track 75.6 -> 48.3 mm
- net OLED_MOSI: track 106.2 -> 85.2 mm, vias 4 -> 2
- net OLED_SCK: track 105.2 -> 85.7 mm, vias 4 -> 2
- net OLED_CS: track 59.4 -> 42.2 mm, vias 2 -> 0
- net OLED_DC: track 58.8 -> 42.7 mm, vias 2 -> 0
- net nRF24_IRQ: track 36.9 -> 21.5 mm
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- added copper zone on B.Cu, net GND
- added copper zone on F.Cu, net GND

Commit message: produkcja v6
Parts:
- added R14: 100K, Resistor_SMD:R_0402_1005Metric, F.Cu at (130.2, 104.2)
- added R32: 100K, Resistor_SMD:R_0402_1005Metric, F.Cu at (130.1, 106.5)
- added R33: 10K, Resistor_SMD:R_0402_1005Metric, F.Cu at (133.7, 100.3)
- added U3: ~, Package_TO_SOT_SMD:TSOT-23-6_HandSoldering, F.Cu at (134.3, 105.2)
- C3: footprint Resistor_SMD:R_1206_3216Metric -> Capacitor_SMD:C_0805_2012Metric
- J6: value Conn_01x02_Pin -> PRT-14417; footprint Connector_JST:JST_PH_S2B-PH-SM4-TB_1x02-1MP_P2.00mm_Horizontal -> BM04B-SRSS-TB_LF__SN_:SPARKFUN_PRT-14417
- moved J6 1.53 mm to (176.3, 99.1)
- renumbered J3 to +, J4 to -
Connections:
- CPU1 pad 24: unconnected-(CPU1-PA1-Pad24) -> GPS_ON_OFF
- J6 pad 1: GND -> SW_IN
- R27 pad 2: SW_OUT -> Net-(R27-Pad2)
Routing:
- net SW_OUT: track 48.3 -> 28.6 mm
- net Net-(R27-Pad2): track 0.00 -> 16.4 mm
- net GPS_ON_OFF: track 0.00 -> 8.75 mm
- net Net-(R14-Pad1): track 0.00 -> 7.96 mm, vias 0 -> 2
- net Net-(R32-Pad2): track 0.00 -> 7.41 mm
- net Net-(RADIO1-~{CSN}): track 22.0 -> 17.1 mm
- net GND: track 196.9 -> 199.4 mm, vias 24 -> 26
- net +3V3: track 249.8 -> 248.1 mm
- net SW_IN: track 104.7 -> 106.2 mm
- net SWDIO: track 16.4 -> 15.2 mm
- net OLED_RST: track 47.1 -> 46.4 mm
Other:
- board text added: "- BAT +"
- board text added: "GPS"
