File: licznik/licznik.kicad_sch (KiCad schematic)
At the start: 69 parts, among them J1 Conn_01x05_Female, J2 USB_B_Mini, J21 BAT+, J22 BAT-, Q3 AO3401A, U1 AMS1117-3.3, U1 TP4056, U2 LSM6DS3, U3 STM32F407VETx, U4 gps, U5 gyro, U6 oled, Y1 Crystal

Commit message: hardware_2
Parts:
- removed D9: ZMMxx, Diode_SMD:D_MiniMELF, symbol Diode:ZMMxx
- removed R12: 2K, Resistor_SMD:R_0805_2012Metric, symbol Device:R
- removed RESET1: SW_Push, Button_Switch_THT:SW_PUSH_6mm, symbol Switch:SW_Push
- removed U7: ~, symbol sd_card:TF-01A
- added C7, C9: 10uF, Capacitor_Tantalum_SMD:CP_EIA-3216-18_Kemet-A, symbol Device:C_Polarized
- added D3: SM4007, Diode_SMD:D_SOD-123F, symbol Diode:SM4007
- added D4: ZMMxx, Diode_SMD:D_MiniMELF, symbol Diode:ZMMxx
- added H1, H2, H3, H4: MountingHole_Pad, MountingHole:MountingHole_3.2mm_M3, symbol Mechanical:MountingHole_Pad
- added MICRO_SD1: TF-01A, slot_sd:TF-01A, symbol sd_card_slot:TF-01A
- added POWER_BUTTON1: POWER_PB, Connector_PinSocket_2.54mm:PinSocket_2x01_P2.54mm_Vertical, symbol Switch:SW_Push
- added R7: 10K, Resistor_SMD:R_0603_1608Metric, symbol Device:R_Small
- added USER_PB1: USER_PB, TS_1187A-B-A-B:SW_TS-1187A-B-A-B, symbol button:TS-1187A-B-A-B
- C1, C10, C11, C12, C13, C14, C15, C16, C17, C18, C19, C2, C20, C21, C22, C23, C3, C4, C5, C6, C8: footprint Capacitor_SMD:C_0805_2012Metric -> Capacitor_SMD:C_0603_1608Metric
- D2: footprint LED_SMD:LED_0805_2012Metric -> LED_SMD:LED_0603_1608Metric
- F1: footprint Fuse:Fuse_0805_2012Metric -> Diode_SMD:D_SMB
- J2: footprint (none) -> Connector_USB:USB_Mini-B_Wuerth_65100516121_Horizontal
- R1, R10, R11, R12, R13, R14, R15, R16, R18, R2, R24, R3, R4, R5, R8, R9: footprint Resistor_SMD:R_0805_2012Metric -> Resistor_SMD:R_0603_1608Metric
- U1: footprint TO4056:SOP127P600X175-9N -> Package_SO:HSOP-8-1EP_3.9x4.9mm_P1.27mm_EP2.3x2.3mm
Connections:
- net +3V3: now also C9.1, MICRO_SD1.4 (VDD), R7.2
- net +5V: now also D3.2 (A), D4.1 (K), POWER_BUTTON1.2; no longer C3.1, FB1.1, Q3.2 (S), R1.2, U1.3 (VI), U4.1 (VCC)
- net CHRG_SIGNAL: now also U1.7 (~{CHRG})
- net GND: now also C7.2, C9.2, D4.2 (A), H1.1, H2.1, H3.1, H4.1, MICRO_SD1.6 (VSS), MICRO_SD1.MP1 (SHIELD), MICRO_SD1.MP2 (SHIELD), MICRO_SD1.MP3 (SHIELD), MICRO_SD1.MP4 (SHIELD), USER_PB1.A, USER_PB1.B
- net NRST: now also USER_PB1.C, USER_PB1.D
- net SDIO_CMD: now also MICRO_SD1.3 (CMD)
- net SDIO_D0: now also MICRO_SD1.7 (DAT0)
- net SDIO_D1: now also MICRO_SD1.8 (DAT1)
- net SDIO_D2: now also MICRO_SD1.1 (DAT2)
- net SDIO_D3: now also MICRO_SD1.2 (CD/DAT3)
- net SDIO_INSERT_CARD: now also MICRO_SD1.CD1 (CD), R7.1
- net SDIO_SCK: now also MICRO_SD1.5 (CLK)
- new net: FB1.1, POWER_BUTTON1.1
- new net REG_IN: C3.1, C7.1, D3.1 (K), Q3.2 (S), R1.2, U1.3 (VI), U4.1 (VCC)
- no-connect marks 60 -> 63
Other:
- moved on the sheet: C2, C23, C5, R1, R10, R11, R12, R13, R15, R16, U1, U4

Commit message: ulepszony pcb
Parts:
- removed F1: Fuse_Small, Diode_SMD:D_SMB, symbol Device:Fuse_Small
- removed U4: gps, licznik:gp1, symbol gw:gps
- removed U5: gyro, licznik:gy1, symbol gw:gyro
- added J5: BM04B-SRSS-TB_LF__SN_, BM04B-SRSS-TB_LF__SN_:JST_BM04B-SRSS-TB_LF__SN_, symbol BM04B-SRSS-TB_LF__SN_:BM04B-SRSS-TB_LF__SN_
Connections:
- net GND: now also J5.1, J5.S1 (SHIELD), J5.S2 (SHIELD)
- net GPS_UART_RX: now also J5.4
- net GPS_UART_TX: now also J5.3
- net REG_IN: now also J5.2
- net at FB1.2: now also D1.1 (K)
- no-connect marks 63 -> 57

Commit message: add nRF
Parts:
- removed POWER_BUTTON1: POWER_PB, Connector_PinSocket_2.54mm:PinSocket_2x01_P2.54mm_Vertical, symbol Switch:SW_Push
- added U4: NRF24L01_Breakout, RF_Module:nRF24L01_Breakout, symbol RF:NRF24L01_Breakout
Connections:
- net +3V3: now also J2.4 (ID), U4.2 (VCC); no longer C5.1, C9.1, U1.2 (VO)
- net +5V: now also FB1.1
- net GND: now also U4.1 (GND); no longer J2.4 (ID)
- net OLED_MISO: now also U4.7 (MISO)
- net OLED_MOSI: now also U4.6 (MOSI)
- net OLED_SCK: now also U4.5 (SCK)
- net PB_OK: no longer J2.2 (D-)
- net nRF24_CE: now reaches U3.67 (PA8)
- net nRF24_CE: now also U4.3 (CE)
- net nRF24_IRQ: now reaches U3.68 (PA9)
- net nRF24_IRQ: now also U4.8 (IRQ)
- net nRF24_CNS: now reaches U3.69 (PA10)
- net nRF24_CNS: now also U4.4 (~{CSN})
- new net REG_OUT: C5.1, C9.1, J2.2 (D-), U1.2 (VO)
- no-connect marks 57 -> 53
Other:
- moved on the sheet: C10, C23, C8, J1, J5, MICRO_SD1, R10, R11, R12, R13, R15, R16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

Commit message: wip
Parts:
- removed C3, C5: 100nF, Capacitor_SMD:C_0603_1608Metric, symbol Device:C_Small
- removed D1: LED, LED_SMD:LED_0603_1608Metric, symbol Device:LED
- removed JUMPERS1: jump, Connector_PinHeader_1.00mm:PinHeader_1x02_P1.00mm_Vertical, symbol Connector:Conn_01x02_Pin
- removed PB_UP1: SW_Push, Connector_PinSocket_2.54mm:PinSocket_2x01_P2.54mm_Vertical, symbol Switch:SW_Push
- removed R1: 2K, Resistor_SMD:R_0603_1608Metric, symbol Device:R
- removed R2, R4: 10K, Resistor_SMD:R_0603_1608Metric, symbol Device:R_Small
- added JP1: JP_MOSI, symbol Jumper:Jumper_2_Bridged
- added JP2: JP_MISO, symbol Jumper:Jumper_2_Bridged
- added JP3: JP_SCK, symbol Jumper:Jumper_2_Bridged
- added JP4: JP_CNS, symbol Jumper:Jumper_2_Bridged
- added JP5: JP_CE, symbol Jumper:Jumper_2_Bridged
- added JP_CE1: JP_IRQ, symbol Jumper:Jumper_2_Bridged
- GPS1: renamed from J5; value BM04B-SRSS-TB_LF__SN_ -> GPS
- RADIO1: renamed from U4; footprint RF_Module:nRF24L01_Breakout -> nRF:NRF24L01-SMD_mini
- USER_PB1: value USER_PB -> RESET
- renumbered U3 to CPU1
Connections:
- net +3V3: no longer R12.2
- net +5V: now also R12.2
- net OLED_MISO: now also JP2.1 (A); no longer RADIO1.7 (MISO)
- net OLED_MOSI: now also JP1.1 (A); no longer RADIO1.6 (MOSI)
- net OLED_SCK: now also JP3.1 (A); no longer RADIO1.5 (SCK)
- net nRF24_CE: now also JP5.1 (A); no longer RADIO1.3 (CE)
- net nRF24_CNS: now also JP4.1 (A); no longer RADIO1.4 (~{CSN})
- net nRF24_IRQ: now also JP_CE1.1 (A); no longer RADIO1.8 (IRQ)
- new net: JP5.2 (B), RADIO1.3 (CE)
- new net: JP_CE1.2 (B), RADIO1.8 (IRQ)
- new net: JP4.2 (B), RADIO1.4 (~{CSN})
- new net: JP3.2 (B), RADIO1.5 (SCK)
- new net: JP1.2 (B), RADIO1.6 (MOSI)
- new net: JP2.2 (B), RADIO1.7 (MISO)
Other:
- moved on the sheet: C2, GPS1, H1, H2, H3, H4, R1, RADIO1, USER_PB1

Commit message: przed poprawkami
Parts:
- removed GPS1: GPS, BM04B-SRSS-TB_LF__SN_:JST_BM04B-SRSS-TB_LF__SN_, symbol BM04B-SRSS-TB_LF__SN_:BM04B-SRSS-TB_LF__SN_
- removed JP1: JP_MOSI, symbol Jumper:Jumper_2_Bridged
- removed JP2: JP_MISO, symbol Jumper:Jumper_2_Bridged
- removed JP3: JP_SCK, symbol Jumper:Jumper_2_Bridged
- removed JP4: JP_CNS, symbol Jumper:Jumper_2_Bridged
- removed JP5: JP_CE, symbol Jumper:Jumper_2_Bridged
- removed JP_CE1: JP_IRQ, symbol Jumper:Jumper_2_Bridged
- added J5: PRT-14417, BM04B-SRSS-TB_LF__SN_:SPARKFUN_PRT-14417, symbol PRT-14417:PRT-14417
- added J6: Conn_01x02_Pin, Connector_JST:JST_PH_S2B-PH-SM4-TB_1x02-1MP_P2.00mm_Horizontal, symbol Connector:Conn_01x02_Pin
- added R17, R19, R2, R22, R24, R25, R26, R27, R28, R29, R4: 0R, Resistor_SMD:R_0603_1608Metric, symbol Device:R_Small
Connections:
- net +3V3: now also C5.1, C9.1, U1.2 (VO), R25.1; no longer J2.4 (ID), RADIO1.2 (VCC)
- net GND: now also J6.1 (Pin_1), R29.2
- net GPS_UART_RX: now also R26.2
- net GPS_UART_TX: now also R28.2
- net OLED_MISO: now also R4.2
- net OLED_MOSI: now also R2.2
- net OLED_SCK: now also R17.2
- net VBAT: now also J6.2 (Pin_2)
- net nRF24_CE: now also R22.2
- net nRF24_CNS: now also R19.2
- net nRF24_IRQ: now also R24.2
- net at RADIO1.3 (CE): now also R22.1
- net at RADIO1.8 (IRQ): now also R24.1
- net at RADIO1.4 (~{CSN}): now also R19.1
- net at RADIO1.5 (SCK): now also R17.1
- net at RADIO1.6 (MOSI): now also R2.1
- net at RADIO1.7 (MISO): now also R4.1
- net REG_IN renamed SW_OUT
- net SW_OUT: now also J2.4 (ID), R27.2; no longer D3.1 (K), Q3.2 (S)
- removed net REG_OUT: C5.1, C9.1, J2.2 (D-), U1.2 (VO)
- new net: R25.2, RADIO1.2 (VCC)
- new net: J5.2, R27.1
- new net: J5.1, R29.1
- new net: J5.3, R28.1
- new net: J5.4, R26.1
- new net SW_IN: D3.1 (K), J2.2 (D-), Q3.2 (S)
Other:
- moved on the sheet: C3, C5, C7, C9, D3, D4, Q3, R24, U1

Commit message: proukcja v5
Parts:
- removed C2: 100nF, Capacitor_SMD:C_0603_1608Metric, symbol Device:C_Small
- removed C7, C9: 10uF, Capacitor_Tantalum_SMD:CP_EIA-3216-18_Kemet-A, symbol Device:C_Polarized
- removed D3: SM4007, Diode_SMD:D_SOD-123F, symbol Diode:SM4007
- removed D4: ZMMxx, Diode_SMD:D_MiniMELF, symbol Diode:ZMMxx
- removed Q3: AO3401A, Package_TO_SOT_SMD:SOT-23, symbol Transistor_FET:AO3401A
- removed R14: 0R, Resistor_SMD:R_0603_1608Metric, symbol Device:R_Small
- removed R24: 10K, Resistor_SMD:R_0603_1608Metric, symbol Device:R
- removed U1: AMS1117-3.3, Package_TO_SOT_SMD:SOT-223-3_TabPin2, symbol Regulator_Linear:AMS1117-3.3
- removed USER_PB1: RESET, TS_1187A-B-A-B:SW_TS-1187A-B-A-B, symbol button:TS-1187A-B-A-B
- added C2: 10uF, Capacitor_SMD:C_0603_1608Metric, symbol Device:C
- added L1: 10uH, Inductor_SMD:L_0805_2012Metric, symbol Device:L
- added R23: 510K, Resistor_SMD:R_0603_1608Metric, symbol Device:R_Small
- added R30: 120K, Resistor_SMD:R_0603_1608Metric, symbol Device:R_Small
- added R31: 200K, Resistor_SMD:R_0603_1608Metric, symbol Device:R_Small
- added U1: MCP1601-I_MS, Package_DFN_QFN:TDFN-8-1EP_3x2mm_P0.5mm_EP1.3x1.4mm, symbol mcp:MCP1601-I_MS
- C1, C11, C12, C13, C14, C15, C16, C17, C18, C19, C20, C21, C22, C6: footprint Capacitor_SMD:C_0603_1608Metric -> Capacitor_SMD:C_0402_1005Metric
- C3: value 22uF -> 47pF; footprint Capacitor_SMD:C_0603_1608Metric -> Resistor_SMD:R_1206_3216Metric
- C5: value 22uF -> 10uF
- R1: value 10K -> 50K
- R18, R8, R9: footprint Resistor_SMD:R_0603_1608Metric -> Resistor_SMD:R_0402_1005Metric
Connections:
- net VBAT is gone; now on net SW_IN: C4.1, J21.1 (Pin_1), J6.2 (Pin_2), U1.5 (BAT)
- net +3V3: now also C3.1, R12.2, L1.2, R23.2, U1.6 (VOUT); no longer R1.2
- net +5V: no longer R12.2
- net GND: now also C2.2, R31.1, U1.4 (AGND), U1.5 (SYNC/PWM), U1.7 (PGND); no longer C3.2
- net NRST: no longer R1.1
- net PB_DOWN: now also R1.1; no longer C4.1, J2.3 (D+), R3.1
- net SW_OUT: now also C2.1, U1.1 (VIN), U1.2 (~{SHDN}); no longer C3.1
- net at R5.1: now also D2.2 (A)
- new net: L1.1, U1.8 (LX)
- new net: R23.1, R30.2
- new net: C3.2, R30.1, R31.2, U1.3 (FB)
- new net PUSH_DOWN_IN: C4.1, J2.3 (D+), R1.2, R3.1
- no-connect marks 53 -> 52
Other:
- moved on the sheet: C1, C4, C6, D1, D2, FB1, J1, J2, J21, J22, J6, R12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

Commit message: produkcja v6
Parts:
- removed J6: Conn_01x02_Pin, Connector_JST:JST_PH_S2B-PH-SM4-TB_1x02-1MP_P2.00mm_Horizontal, symbol Connector:Conn_01x02_Pin
- added J6: PRT-14417, BM04B-SRSS-TB_LF__SN_:SPARKFUN_PRT-14417, symbol PRT-14417:PRT-14417
- added R14, R32: 100K, Resistor_SMD:R_0402_1005Metric, symbol Device:R_Small
- added R33: 10K, Resistor_SMD:R_0402_1005Metric, symbol Device:R_Small
- added U3: ~, Package_TO_SOT_SMD:TSOT-23-6_HandSoldering, symbol SIL2308:SIL2308
- C3: footprint Resistor_SMD:R_1206_3216Metric -> Capacitor_SMD:C_0805_2012Metric
Connections:
- net GND: now also J6.3, J6.4, R14.2, U3.5
- net SW_IN: now also J6.1, J6.2
- net SW_OUT: now also R32.1, U3.2; no longer R27.2
- net GPS_ON_OFF: now reaches CPU1.24 (PA1)
- net GPS_ON_OFF: now also R33.1
- new net: R32.2, U3.3, U3.6
- new net: R14.1, R33.2, U3.1
- new net: R27.2, U3.4
- no-connect marks 52 -> 50
Other:
- moved on the sheet: J5, R26, R27, R28, R29
